File: PCB/Digital.kicad_sch (KiCad schematic)
At the start: 16 parts, among them IC1 MAX3051ESA+, J2 ICSP, J3 DE9_Plug_MountingHoles, J4 Conn_Coaxial, J5 DE9_Plug_MountingHoles, U1 PIC18F2580T-I/SO, Y2 ABLS-8.000MHZ-B2-T

Commit message: Add files via upload
Parts:
- C5, C6: value C -> 22p
Other:
- note added: "CRISTALL OSCIL-LADOR"
Changed lines of the file:
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@@
+		)
+	)
+	(text "CRISTALL OSCIL-LADOR"
+		(exclude_from_sim no)
+		(at 22.352 90.424 0)
+		(effects
+			(font
+				(size 2.032 2.032)
+				(thickness 0.6)
+				(bold yes)
+			)
+			(justify left bottom)
 		)
 	)
@@
 	)
 	(junction
+		(at 43.18 66.04)
+		(diameter 0)
+		(color 0 0 0 0)
+	)
+	(junction
 		(at 25.4 66.04)
 		(diameter 0)
@@
 	)
 	(junction
-		(at 43.18 66.04)
-		(diameter 0)
-		(color 0 0 0 0)
-	)
-	(junction
 		(at 46.99 34.29)
 		(diameter 0)
@@
 	(wire
 		(pts
-			(xy 50.8 59.69) (xy 25.4 59.69)
-		)
-		(stroke
-			(width 0)
-			(type default)
-		)
-	)
-	(wire
-		(pts
 			(xy 46.99 34.29) (xy 46.99 35.56)
 		)
@@
 	(wire
 		(pts
-			(xy 43.18 152.4) (xy 31.75 152.4)
-		)
-		(stroke
-			(width 0)
-			(type default)
-		)
-	)
-	(wire
-		(pts
 			(xy 68.58 59.69) (xy 71.12 59.69)
 		)
@@
 	(wire
 		(pts
-			(xy 71.12 52.07) (xy 44.45 52.07)
+			(xy 71.12 52.07) (xy 15.24 52.07)
 		)
 		(stroke
@@
 	(wire
 		(pts
-			(xy 44.45 52.07) (xy 44.45 53.34)
+			(xy 15.24 52.07) (xy 15.24 53.34)
 		)
 		(stroke
@@
 	(wire
 		(pts
-			(xy 71.12 57.15) (xy 53.34 57.15)
-		)
-		(stroke
-			(width 0)
-			(type default)
-		)
-	)
-	(wire
-		(pts
 			(xy 68.58 41.91) (xy 71.12 41.91)
 		)
@@
 	(wire
 		(pts
+			(xy 43.18 57.15) (xy 71.12 57.15)
+		)
+		(stroke
+			(width 0)
+			(type default)
+		)
+	)
+	(wire
+		(pts
 			(xy 93.98 148.59) (xy 93.98 152.4)
 		)
@@
 	(wire
 		(pts
-			(xy 31.75 152.4) (xy 31.75 147.32)
-		)
-		(stroke
-			(width 0)
-			(type default)
-		)
-	)
-	(wire
-		(pts
 			(xy 194.31 116.84) (xy 196.85 116.84)
 		)
@@
 	(wire
 		(pts
+			(xy 25.4 54.61) (xy 71.12 54.61)
+		)
+		(stroke
+			(width 0)
+			(type default)
+		)
+	)
+	(wire
+		(pts
 			(xy 67.31 62.23) (xy 71.12 62.23)
 		)
@@
 	(wire
 		(pts
+			(xy 25.4 54.61) (xy 25.4 66.04)
+		)
+		(stroke
+			(width 0)
+			(type default)
+		)
+	)
+	(wire
+		(pts
 			(xy 88.9 158.75) (xy 95.25 158.75)
 		)
@@
 	(wire
 		(pts
-			(xy 31.75 147.32) (xy 24.13 147.32)
+			(xy 24.13 152.4) (xy 43.18 152.4)
 		)
 		(stroke
@@
 	(wire
 		(pts
-			(xy 25.4 59.69) (xy 25.4 66.04)
-		)
-		(stroke
-			(width 0)
-			(type default)
-		)
-	)
-	(wire
-		(pts
-			(xy 71.12 54.61) (xy 50.8 54.61)
-		)
-		(stroke
-			(width 0)
-			(type default)
-		)
-	)
-	(wire
-		(pts
 			(xy 80.01 148.59) (xy 88.9 148.59)
 		)
@@
 	(wire
 		(pts
+			(xy 43.18 57.15) (xy 43.18 66.04)
+		)
+		(stroke
+			(width 0)
+			(type default)
+		)
+	)
+	(wire
+		(pts
 			(xy 246.38 40.64) (xy 246.38 44.45)
 		)
@@
 	(wire
 		(pts
-			(xy 50.8 54.61) (xy 50.8 59.69)
-		)
-		(stroke
-			(width 0)
-			(type default)
-		)
-	)
-	(wire
-		(pts
-			(xy 53.34 66.04) (xy 43.18 66.04)
-		)
-		(stroke
-			(width 0)
-			(type default)
-		)
-	)
-	(wire
-		(pts
 			(xy 254 124.46) (xy 254 128.27)
 		)
@@
 	(wire
 		(pts
-			(xy 53.34 57.15) (xy 53.34 66.04)
-		)
-		(stroke
-			(width 0)
-			(type default)
-		)
-	)
-	(wire
-		(pts
-			(xy 24.13 147.32) (xy 24.13 154.94)
+			(xy 24.13 152.4) (xy 24.13 154.94)
 		)
 		(stroke
@@
 			)
 		)
-		(property "Value" "C"
+		(property "Value" "22p"
 			(at 29.21 73.6599 0)
 			(effects
@@
 	(symbol
 		(lib_id "power:GND")
-		(at 44.45 53.34 0)
+		(at 15.24 53.34 0)
 		(unit 1)
 		(exclude_from_sim no)
@@
 		(dnp no)
 		(property "Reference" "#PWR030"
-			(at 44.45 59.69 0)
+			(at 15.24 59.69 0)
 			(effects
 				(font
@@
 		)
 		(property "Value" "GND"
-			(at 47.498 56.134 0)
+			(at 18.288 56.134 0)
 			(effects
 				(font
@@
 		)
 		(property "Footprint" ""
-			(at 44.45 53.34 0)
+			(at 15.24 53.34 0)
 			(effects
 				(font
@@
 		)
 		(property "Datasheet" ""
-			(at 44.45 53.34 0)
+			(at 15.24 53.34 0)
 			(effects
 				(font
@@
 		)
 		(property "Description" ""
-			(at 44.45 53.34 0)
+			(at 15.24 53.34 0)
 			(effects
 				(font
@@
 			)
 		)
-		(property "Value" "C"
+		(property "Value" "22p"
 			(at 46.99 73.6599 0)
 			(effects

Commit message: Update Digital.kicad_sch
Parts:
- removed C8: 100n, symbol Device:C
- added C1: 100n, symbol Device:C
Connections:
- net +5V: now also C1.1
- net GND: now also J3.6, C1.2
- net USART_RX: now also J5.3, U1.17 (RC6/TX/CK); no longer J5.2, U1.18 (RC7/RX/DT)
- net USART_TX: now also J5.2, U1.18 (RC7/RX/DT); no longer J5.3, U1.17 (RC6/TX/CK)
- no-connect marks 23 -> 22
Other:
- moved on the sheet: C5, C6, C7, C9, IC1, J2, J3, J4, J5, R2, R7, R8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

Commit message: Update Digital.kicad_sch
Parts:
- removed J5: DE9_Plug_MountingHoles, Connector_Dsub:DSUB-9_Female_Horizontal_P2.77x2.84mm_EdgePinOffset4.94mm_Housed_MountingHolesOffset7.48mm, symbol Connector:DE9_Plug_MountingHoles
Connections:
- net USART_RX: now also J3.9
- net USART_TX: now also J3.5
- no-connect marks 22 -> 13
Other:
- note added: "BUS CAN / USART"
- note removed: "BUS CAN"
- note removed: "USART"
- moved on the sheet: C7

Commit message: anadido el shdn directo al PIC. Es un pin de alarma térmica del transceiver. El sensor de corriente está mal hay que darle una vuelta
Parts:
- renumbered C1 to C?
Connections:
- net SHDN: now reaches IC1.5 (SHDN)
- net SHDN: now also U1.26 (RB5/KBI1/PGM)
- no-connect marks 13 -> 11
Changed lines of the file:
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@@
 	)
 	(no_connect
-		(at 130.81 67.31)
-	)
-	(no_connect
 		(at 241.3 135.89)
 	)
@@
 		(at 72.39 74.93)
 	)
-	(no_connect
-		(at 227.6649 41.91)
-	)
 	(wire
 		(pts
@@
 	(wire
 		(pts
+			(xy 227.33 41.91) (xy 233.68 41.91)
+		)
+		(stroke
+			(width 0)
+			(type default)
+		)
+	)
+	(wire
+		(pts
 			(xy 44.45 85.09) (xy 72.39 85.09)
 		)
@@
 	(wire
 		(pts
+			(xy 130.81 67.31) (xy 146.05 67.31)
+		)
+		(stroke
+			(width 0)
+			(type default)
+		)
+	)
+	(wire
+		(pts
 			(xy 44.45 93.98) (xy 44.45 96.52)
 		)
@@
 		)
 	)
+	(label "SHDN"
+		(at 228.6 41.91 0)
+		(effects
+			(font
+				(size 1.27 1.27)
+			)
+			(justify left bottom)
+		)
+	)
+	(label "SHDN"
+		(at 137.16 67.31 0)
+		(effects
+			(font
+				(size 1.27 1.27)
+			)
+			(justify left bottom)
+		)
+	)
 	(label "USART_TX"
 		(at 186.69 31.75 0)
@@
 		(dnp no)
 		(fields_autoplaced yes)
-		(property "Reference" "IC?"
+		(property "Reference" "IC1"
 			(at 213.36 34.29 0)
 			(effects
@@
 		(on_board yes)
 		(dnp no)
-		(property "Reference" "C?"
+		(property "Reference" "C6"
 			(at 30.48 99.0599 0)
 			(effects
@@
 		(dnp no)
 		(fields_autoplaced yes)
-		(property "Reference" "#PWR?"
+		(property "Reference" "#PWR052"
 			(at 187.96 144.78 0)
 			(effects
@@
 		(on_board yes)
 		(dnp no)
-		(property "Reference" "#PWR?"
+		(property "Reference" "#PWR030"
 			(at 16.51 87.63 0)
 			(effects
@@
 		(on_board yes)
 		(dnp no)
-		(property "Reference" "R?"
+		(property "Reference" "R2"
 			(at 240.03 41.91 0)
 			(effects
@@
 		(dnp no)
 		(fields_autoplaced yes)
-		(property "Reference" "C?"
+		(property "Reference" "C5"
 			(at 48.26 99.0599 0)
 			(effects
@@
 		(dnp no)
 		(fields_autoplaced yes)
-		(property "Reference" "#PWR?"
+		(property "Reference" "#PWR042"
 			(at 125.73 54.61 0)
 			(effects
@@
 		(on_board yes)
 		(dnp no)
-		(property "Reference" "J?"
+		(property "Reference" "J3"
 			(at 267.97 31.75 90)
 			(effects
@@
 		(dnp no)
 		(fields_autoplaced yes)
-		(property "Reference" "#PWR?"
+		(property "Reference" "#PWR011"
 			(at 44.45 113.03 0)
 			(effects
@@
 		(on_board yes)
 		(dnp no)
-		(property "Reference" "C1"
+		(property "Reference" "C?"
 			(at 175.26 74.9299 0)
 			(effects
@@
 		)
 		(instances
+			(project "puertas"
+				(path "/c96004bd-c0fc-431c-a510-eb1e1a82944f/ddbb6980-9f13-42d8-9727-7a64df9bde6c"
+					(reference "C?")
+					(unit 1)
+				)
+			)
 			(project "Digital"
 				(path "/fabbde56-8e14-4a1d-9ecb-2c0209abd5e9"
@@
 		(dnp no)
 		(fields_autoplaced yes)
-		(property "Reference" "#PWR?"
+		(property "Reference" "#PWR061"
 			(at 257.81 156.21 0)
 			(effects
@@
 		(dnp no)
 		(fields_autoplaced yes)
-		(property "Reference" "J?"
+		(property "Reference" "J2"
 			(at 146.05 43.1799 0)
 			(effects
@@
 		(dnp no)
 		(fields_autoplaced yes)
-		(property "Reference" "C?"
+		(property "Reference" "C7"
 			(at 195.58 50.7999 0)
 			(effects
@@
 		(on_board yes)
 		(dnp no)
-		(property "Reference" "Y?"
+		(property "Reference" "Y2"
 			(at 35.306 100.076 0)
 			(effects
@@
 		(on_board yes)
 		(dnp no)
-		(property "Reference" "#PWR02"
+		(property "Reference" "#PWR0101"
 			(at 171.45 88.9 0)
 			(effects
@@
 		)
 		(instances
+			(project "puertas"
+				(path "/c96004bd-c0fc-431c-a510-eb1e1a82944f/ddbb6980-9f13-42d8-9727-7a64df9bde6c"
+					(reference "#PWR0101")
+					(unit 1)
+				)
+			)
 			(project "Digital"
 				(path "/fabbde56-8e14-4a1d-9ecb-2c0209abd5e9"
@@
 		(on_board yes)
 		(dnp no)
-		(property "Reference" "#PWR01"
+		(property "Reference" "#PWR0102"
 			(at 171.45 72.39 0)
 			(effects
@@
 		)
 		(instances
+			(project "puertas"
+				(path "/c96004bd-c0fc-431c-a510-eb1e1a82944f/ddbb6980-9f13-42d8-9727-7a64df9bde6c"
+					(reference "#PWR0102")
+					(unit 1)
+				)
+			)
 			(project "Digital"
 				(path "/fabbde56-8e14-4a1d-9ecb-2c0209abd5e9"
@@
 		(on_board yes)
 		(dnp no)
-		(property "Reference" "#PWR?"
+		(property "Reference" "#PWR017"
 			(at 24.13 24.13 0)
 			(effects
@@
 		(on_board yes)
 		(dnp no)
-		(property "Reference" "R?"
+		(property "Reference" "R7"
 			(at 32.512 59.69 90)
 			(effects
@@
 		(dnp no)
 		(fields_autoplaced yes)
-		(property "Reference" "#PWR?"
+		(property "Reference" "#PWR018"
 			(at 24.13 78.74 0)
 			(effects
@@
 		(dnp no)
 		(fields_autoplaced yes)
-		(property "Reference" "#PWR?"
+		(property "Reference" "#PWR010"
 			(at 26.67 113.03 0)
 			(effects
@@
 		(dnp no)
 		(fields_autoplaced yes)
-		(property "Reference" "R?"
+		(property "Reference" "R8"
 			(at 26.67 54.6099 0)
 			(effects
@@
 		(dnp no)
 		(fields_autoplaced yes)
-		(property "Reference" "C?"
+		(property "Reference" "C9"
 			(at 27.94 66.0399 0)
 			(effects
@@
 		(dnp no)
 		(fields_autoplaced yes)
-		(property "Reference" "#PWR?"
+		(property "Reference" "#PWR048"
 			(at 196.85 142.24 0)
 			(effects
@@
 		(on_board yes)
 		(dnp no)
-		(property "Reference" "U?"
+		(property "Reference" "U1"
 			(at 98.806 52.832 0)
 			(effects
@@
 		(dnp no)
 		(fields_autoplaced yes)
-		(property "Reference" "U?"
+		(property "Reference" "U6"
 			(at 223.1741 123.19 0)
 			(effects
@@
 		(dnp no)
 		(fields_autoplaced yes)
-		(property "Reference" "J?"
+		(property "Reference" "J4"
 			(at 261.62 129.8331 0)
 			(effects
@@
 		(on_board yes)
 		(dnp no)
-		(property "Reference" "#PWR?"
+		(property "Reference" "#PWR020"
 			(at 191.77 64.77 0)
 			(effects

Commit message: Add files via upload
Parts:
- removed C?: 100n, symbol Device:C
- added C13: 100n, Capacitor_SMD:C_1206_3216Metric, symbol Device:C
- added J1: DE9_Pins_MountingHoles, Connector_Dsub:DSUB-9_Pins_Horizontal_P2.77x2.84mm_EdgePinOffset4.94mm_Housed_MountingHolesOffset4.94mm, symbol Connector:DE9_Pins_MountingHoles
- added J6: Conn_01x03, Connector_PinHeader_2.54mm:PinHeader_1x03_P2.54mm_Vertical, symbol Connector_Generic:Conn_01x03
- added J7: DOOR, Connector_PinHeader_2.54mm:PinHeader_1x05_P2.54mm_Vertical, symbol Connector_Generic:Conn_01x05
- added J8: WINDOW, Connector_PinHeader_2.54mm:PinHeader_1x05_P2.54mm_Vertical, symbol Connector_Generic:Conn_01x05
- added R11, R12, R13, R16, R17: 10k, Capacitor_SMD:C_1206_3216Metric, symbol Device:R
- added S1, S2, S3, S6, S7: 3-1437565-0, 3-1437565-0:314375650, symbol 3-1437565-0:3-1437565-0
- C5, C6: value 22p -> 21p; footprint (none) -> Capacitor_SMD:C_0201_0603Metric
- C7, C9: footprint (none) -> Capacitor_SMD:C_1206_3216Metric
- IC1: footprint SOIC127P600X175-8N -> MAX3051ESA+:SOIC127P600X175-8N
- J2: footprint (none) -> Connector_PinHeader_2.54mm:PinHeader_1x05_P2.54mm_Vertical
- J3: footprint Connector_Dsub:DSUB-9_Female_Horizontal_P2.77x2.84mm_EdgePinOffset4.94mm_Housed_MountingHolesOffset7.48mm -> Connector_Dsub:DSUB-9_Pins_Horizontal_P2.77x2.84mm_EdgePinOffset4.94mm_Housed_MountingHolesOffset4.94mm
- J4: footprint (none) -> Connector_Coaxial:BNC_TEConnectivity_1478035_Horizontal
- R7: footprint (none) -> Resistor_SMD:R_0603_1608Metric
- R8: footprint (none) -> Resistor_SMD:R_1206_3216Metric
- U1: footprint SOIC28-W_MC_MCH -> PIC18F2580T_I_SO:SOIC28-W_MC_MCH
- Y2: value ABLS-8.000MHZ-B2-T -> ABLS; footprint ABLS8000MHZB2T -> ABLS8000MHZB2T:ABLS8000MHZB2T
Connections:
- net +5V: now also C13.1, J7.5 (Pin_5), J8.5 (Pin_5), R11.1, R12.1, R13.1, R16.1, R17.1; no longer U6.7 (VCC)
- net CLOSE: now also J7.3 (Pin_3), R13.2, S3.3 (NO_1), S3.4 (NO_2)
- net DOWN: now also J8.4 (Pin_4), R17.2, S6.3 (NO_1), S6.4 (NO_2)
- net GND: now also J3.3, C13.2, J1.5, J7.1 (Pin_1), J8.1 (Pin_1), S1.1 (COM_1), S1.2 (COM_2), S2.1 (COM_1), S3.1 (COM_1), S3.2 (COM_2), S6.1 (COM_1), S7.1 (COM_1), S7.2 (COM_2)
- net MCLR: now also J6.2 (Pin_2); no longer J2.2 (Pin_2)
- net OPEN: now also J7.4 (Pin_4), R12.2, S2.3 (NO_1), S2.4 (NO_2)
- net UP: now also J8.3 (Pin_3), R16.2, S7.3 (NO_1), S7.4 (NO_2)
- net USART_RX: now also U1.18 (RC7/RX/DT), J1.3; no longer J3.9, U1.17 (RC6/TX/CK)
- net USART_TX: now also U1.17 (RC6/TX/CK), J1.2; no longer J3.5, U1.18 (RC7/RX/DT)
- net +3.3V: now reaches C7.1, IC1.3 (VCC)
- net +3.3V: now also U6.7 (VCC)
- net SHDN: no longer names the net of IC1.5 (SHDN)
- net SHDN: no longer U1.26 (RB5/KBI1/PGM)
- new net MAN_MCLR: J6.3 (Pin_3), R11.2, S1.3 (NO_1), S1.4 (NO_2)
- new net PROG_MCLR: J2.2 (Pin_2), J6.1 (Pin_1)
- no-connect marks 11 -> 23
Other:
- note added: "BUS CAN"
- note added: "BUS USART"
- note added: "Botonera"
- note added: "Botonera puerta dentro de la PCB y de conexión externa"
- note added: "Botonera ventana dentro de la PCB y de conexión externa"
- note added: "CRISTALL OSCILADOR"
- note added: "Conector de programación"
- note added: "RESET MANUAL"
- note removed: "BUS CAN / USART"
- note removed: "CRISTALL OSCIL-LADOR"
- note removed: "Connector de programació."
- moved on the sheet: C5, C6, C7, C9, IC1, J2, J3, J4, R2, R7, R8, U1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

Commit message: esquemático  v2
Connections:
- net GND: now also S2.2 (COM_2), S6.2 (COM_2)
Other:
- moved on the sheet: C13, C5, C6, C7, C9, IC1, J1, J2, J3, J4, J6, J7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
