File: PCB/Regulador.kicad_sch (KiCad schematic)
At the start: 14 parts, among them J5 BAT_CONN, U3 LT1121IST-3.3-TRPBF, U5 LM1117DT-5.0

Commit message: Update PCB
Parts:
- U3: footprint Package_TO_SOT_SMD:SOT-223-3_TabPin2 -> LT1121IST-3.3-TRPBF:SOT-223_ST_LIT
Connections:
- net GND: now also U3.4 (GND)
Other:
- title: (none) -> Reguladores de tensión 
- moved on the sheet: C8
Changed lines of the file:
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@@
 	(generator_version "9.0")
 	(paper "A4")
+	(title_block
+		(title "Reguladores de tensión ")
+		(rev "4/4")
+	)
 	(text "SEPARACIÓN DE GNDs\n"
 		(exclude_from_sim no)
@@
 	)
 	(junction
-		(at 73.66 127)
+		(at 228.6 83.82)
 		(diameter 0)
 		(color 0 0 0 0)
 	)
 	(junction
-		(at 203.2 71.12)
+		(at 73.66 127)
 		(diameter 0)
 		(color 0 0 0 0)
@@
 	)
 	(junction
-		(at 226.06 83.82)
-		(diameter 0)
-		(color 0 0 0 0)
-	)
-	(junction
 		(at 147.32 66.04)
 		(diameter 0)
@@
 	)
 	(junction
-		(at 203.2 83.82)
+		(at 200.66 83.82)
 		(diameter 0)
 		(color 0 0 0 0)
@@
 	)
 	(junction
+		(at 200.66 71.12)
+		(diameter 0)
+		(color 0 0 0 0)
+	)
+	(junction
 		(at 154.94 66.04)
 		(diameter 0)
@@
 	)
 	(junction
+		(at 205.74 83.82)
+		(diameter 0)
+		(color 0 0 0 0)
+	)
+	(junction
 		(at 142.24 66.04)
 		(diameter 0)
@@
 	(wire
 		(pts
-			(xy 226.06 73.66) (xy 226.06 83.82)
-		)
-		(stroke
-			(width 0)
-			(type default)
-		)
-	)
-	(wire
-		(pts
 			(xy 101.6 66.04) (xy 111.76 66.04)
 		)
@@
 	(wire
 		(pts
-			(xy 203.2 68.58) (xy 203.2 71.12)
+			(xy 200.66 68.58) (xy 200.66 71.12)
+		)
+		(stroke
+			(width 0)
+			(type default)
+		)
+	)
+	(wire
+		(pts
+			(xy 200.66 71.12) (xy 208.28 71.12)
 		)
 		(stroke
@@
 	(wire
 		(pts
+			(xy 226.06 73.66) (xy 228.6 73.66)
+		)
+		(stroke
+			(width 0)
+			(type default)
+		)
+	)
+	(wire
+		(pts
 			(xy 91.44 76.2) (xy 91.44 78.74)
 		)
@@
 	(wire
 		(pts
-			(xy 226.06 83.82) (xy 233.68 83.82)
+			(xy 228.6 73.66) (xy 228.6 83.82)
 		)
 		(stroke
@@
 	(wire
 		(pts
-			(xy 203.2 71.12) (xy 208.28 71.12)
+			(xy 205.74 83.82) (xy 228.6 83.82)
 		)
 		(stroke
@@
 	(wire
 		(pts
+			(xy 228.6 83.82) (xy 233.68 83.82)
+		)
+		(stroke
+			(width 0)
+			(type default)
+		)
+	)
+	(wire
+		(pts
+			(xy 200.66 83.82) (xy 205.74 83.82)
+		)
+		(stroke
+			(width 0)
+			(type default)
+		)
+	)
+	(wire
+		(pts
 			(xy 233.68 71.12) (xy 233.68 73.66)
 		)
@@
 	(wire
 		(pts
+			(xy 208.28 73.66) (xy 205.74 73.66)
+		)
+		(stroke
+			(width 0)
+			(type default)
+		)
+	)
+	(wire
+		(pts
 			(xy 142.24 66.04) (xy 142.24 68.58)
 		)
@@
 	(wire
 		(pts
-			(xy 203.2 71.12) (xy 203.2 73.66)
+			(xy 200.66 71.12) (xy 200.66 72.39)
 		)
 		(stroke
@@
 	(wire
 		(pts
-			(xy 203.2 83.82) (xy 226.06 83.82)
-		)
-		(stroke
-			(width 0)
-			(type default)
-		)
-	)
-	(wire
-		(pts
-			(xy 203.2 81.28) (xy 203.2 83.82)
+			(xy 205.74 73.66) (xy 205.74 83.82)
+		)
+		(stroke
+			(width 0)
+			(type default)
+		)
+	)
+	(wire
+		(pts
+			(xy 200.66 80.01) (xy 200.66 83.82)
 		)
 		(stroke
@@
 		(lib_name "+5V_1")
 		(lib_id "power:+5V")
-		(at 203.2 68.58 0)
+		(at 200.66 68.58 0)
 		(unit 1)
 		(exclude_from_sim no)
@@
 		(fields_autoplaced yes)
 		(property "Reference" "#PWR014"
-			(at 203.2 72.39 0)
+			(at 200.66 72.39 0)
 			(effects
 				(font
@@
 		)
 		(property "Value" "+5V"
-			(at 203.2 63.5 0)
+			(at 200.66 63.5 0)
 			(effects
 				(font
@@
 		)
 		(property "Footprint" ""
-			(at 203.2 68.58 0)
+			(at 200.66 68.58 0)
 			(effects
 				(font
@@
 		)
 		(property "Datasheet" ""
-			(at 203.2 68.58 0)
+			(at 200.66 68.58 0)
 			(effects
 				(font
@@
 		)
 		(property "Description" "Power symbol creates a global label with name \"+5V\""
-			(at 203.2 68.58 0)
+			(at 200.66 68.58 0)
 			(effects
 				(font
@@
 		(lib_name "GND_2")
 		(lib_id "power:GND")
-		(at 203.2 83.82 0)
+		(at 200.66 83.82 0)
 		(unit 1)
 		(exclude_from_sim no)
@@
 		(fields_autoplaced yes)
 		(property "Reference" "#PWR013"
-			(at 203.2 90.17 0)
+			(at 200.66 90.17 0)
 			(effects
 				(font
@@
 		)
 		(property "Value" "GND"
-			(at 203.2 88.9 0)
+			(at 200.66 88.9 0)
 			(effects
 				(font
@@
 		)
 		(property "Footprint" ""
-			(at 203.2 83.82 0)
+			(at 200.66 83.82 0)
 			(effects
 				(font
@@
 		)
 		(property "Datasheet" ""
-			(at 203.2 83.82 0)
+			(at 200.66 83.82 0)
 			(effects
 				(font
@@
 		)
 		(property "Description" "Power symbol creates a global label with name \"GND\" , ground"
-			(at 203.2 83.82 0)
+			(at 200.66 83.82 0)
 			(effects
 				(font
@@
 			)
 		)
-		(property "Footprint" "Package_TO_SOT_SMD:SOT-223-3_TabPin2"
+		(property "Footprint" "LT1121IST-3.3-TRPBF:SOT-223_ST_LIT"
 			(at 198.12 71.12 0)
 			(effects
@@
 		)
 		(pin "2"
+		)
+		(pin "4"
 		)
 		(instances
@@
 	(symbol
 		(lib_id "Device:C")
-		(at 203.2 77.47 0)
+		(at 200.66 76.2 0)
 		(unit 1)
 		(exclude_from_sim no)
@@
 		(dnp no)
 		(property "Reference" "C8"
-			(at 203.708 74.93 0)
+			(at 198.12 73.66 0)
 			(effects
 				(font
@@
 		)
 		(property "Value" "100n"
-			(at 204.47 79.756 0)
+			(at 195.58 78.74 0)
 			(effects
 				(font
@@
 		)
 		(property "Footprint" "Capacitor_SMD:C_1206_3216Metric"
-			(at 204.1652 81.28 0)
+			(at 201.6252 80.01 0)
 			(effects
 				(font
@@
 		)
 		(property "Datasheet" "~"
-			(at 203.2 77.47 0)
+			(at 200.66 76.2 0)
 			(effects
 				(font
@@
 		)
 		(property "Description" ""
-			(at 203.2 77.47 0)
-			(effects
-				(font
+			(at 200.66 76.2 0)
+			(effects
+				(font
