File: PCB/puertas.kicad_sch (KiCad schematic)
At the start: 0 parts

Commit message: Update PCB
Other:
- title: (none) -> Puertas
Changed lines of the file:
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@@
 	(generator_version "9.0")
 	(paper "A4")
+	(title_block
+		(title "Puertas")
+	)
 	(text "PUERTAS EDD\n"
 		(exclude_from_sim no)
